File: x32promicro.kicad_pcb (KiCad board)
At the start: 2 copper layers, 17.8 x 33 mm, 29 parts, among them J1 USB2.0_C_v3, J2 ProMicro-LeftPin-NoGND, J3 ProMicro-RightPin, SW1 SW_Push, SW2 SW_Push, U1 STM32V103C8T6, U2 AMS1117-3.3, Y1 32.768k, Y2 8M

Commit message: x32micro
Parts:
- renumbered C4 to C1, C7 to C2, C8 to C3, C5 to C4, C2 to C5, C1 to C6, C3 to C7, C6 to C8, R5 to R1, R4 to R2, R1 to R3, R3 to R4, R7 to R5, R8 to R6, R6 to R7, SW2 to SW1, SW1 to SW2, U2 to U1, U1 to U2

Commit message: 少しシルクが欠けている
Other:
- board text added: "v1.1.2"
- board text removed: "+"
- board text removed: "v1.1.1"
Changed lines of the file:
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@@
     (property "ki_keywords" "cap capacitor")
     (attr smd)
-    (fp_text reference "C8" (at -0.1375 -1.2) (layer "B.SilkS")
+    (fp_text reference "C8" (at -2.7225 0.478) (layer "B.SilkS")
         (effects (font (size 0.8 0.8) (thickness 0.12)) (justify mirror))
     )
@@
   (gr_arc (start 101.279026 133.010974) (mid 100.381 132.639) (end 100.009026 131.740974)
     (stroke (width 0.1) (type solid)) (layer "Edge.Cuts"))
-  (gr_text "v1.1.1" (at 112.7 109) (layer "B.SilkS")
+  (gr_text "v1.1.2" (at 112.7 109) (layer "B.SilkS")
     (effects (font (face "Roboto") (size 1.4 1.4) (thickness 0.15)) (justify mirror))
-    (render_cache "v1.1.1" 0
+    (render_cache "v1.1.2" 0
       (polygon
         (pts
@@
       (polygon
         (pts
-          (xy 110.456873 108.180413)          (xy 110.456873 109.581)          (xy 110.633998 109.581)          (xy 110.633998 108.401307)
-          (xy 110.995086 108.531586)          (xy 110.995086 108.3719)          (xy 110.48457 108.180413)
+          (xy 110.130662 109.436017)          (xy 110.130662 109.581)          (xy 111.049797 109.581)          (xy 111.049797 109.45414)
+          (xy 110.573132 108.933023)          (xy 110.558688 108.916865)          (xy 110.544848 108.901132)          (xy 110.531611 108.885823)
+          (xy 110.518978 108.87094)          (xy 110.506948 108.856481)          (xy 110.495523 108.842447)          (xy 110.484701 108.828837)
+          (xy 110.474483 108.815652)          (xy 110.464868 108.802892)          (xy 110.455858 108.790557)          (xy 110.447451 108.778647)
+          (xy 110.439648 108.767161)          (xy 110.429075 108.750729)          (xy 110.419861 108.735252)          (xy 110.414472 108.725466)
+          (xy 110.407139 108.711034)          (xy 110.400528 108.69659)          (xy 110.394637 108.682135)          (xy 110.389468 108.667667)
+          (xy 110.38502 108.653187)          (xy 110.381293 108.638696)          (xy 110.378288 108.624192)          (xy 110.376004 108.609676)
+          (xy 110.374441 108.595148)          (xy 110.3736 108.580609)          (xy 110.37344 108.570909)          (xy 110.373998 108.552187)
+          (xy 110.375675 108.533975)          (xy 110.37847 108.516275)          (xy 110.382383 108.499085)          (xy 110.387414 108.482407)
+          (xy 110.393563 108.466239)          (xy 110.40083 108.450582)          (xy 110.409215 108.435436)          (xy 110.418718 108.420801)
+          (xy 110.429339 108.406677)          (xy 110.43704 108.397545)          (xy 110.449425 108.384651)          (xy 110.46273 108.373026)
+          (xy 110.476954 108.362668)          (xy 110.492098 108.353579)          (xy 110.508162 108.345758)          (xy 110.525145 108.339206)
+          (xy 110.543047 108.333921)          (xy 110.56187 108.329905)          (xy 110.581612 108.327157)          (xy 110.595284 108.32603)
+          (xy 110.609365 108.325466)          (xy 110.616559 108.325396)          (xy 110.633764 108.325703)          (xy 110.650416 108.326625)
+          (xy 110.666515 108.328161)          (xy 110.682062 108.330311)          (xy 110.697055 108.333076)          (xy 110.711495 108.336455)
+          (xy 110.725383 108.340449)          (xy 110.738717 108.345057)          (xy 110.751498 108.35028)          (xy 110.769633 108.359266)
+          (xy 110.786524 108.369634)          (xy 110.802171 108.381385)          (xy 110.816574 108.394519)          (xy 110.825484 108.404042)
+          (xy 110.837828 108.419179)          (xy 110.848958 108.435097)          (xy 110.858873 108.451797)          (xy 110.867575 108.469278)
+          (xy 110.875062 108.48754)          (xy 110.881335 108.506584)          (xy 110.886394 108.526409)          (xy 110.889092 108.54006)
+          (xy 110.891251 108.554058)          (xy 110.89287 108.568404)          (xy 110.893949 108.583096)          (xy 110.894489 108.598136)
+          (xy 110.894556 108.605787)          (xy 111.071681 108.605787)          (xy 111.071228 108.584139)          (xy 111.06987 108.562879)
+          (xy 111.067606 108.542006)          (xy 111.064436 108.52152)          (xy 111.060361 108.501422)          (xy 111.05538 108.481711)
+          (xy 111.049494 108.462387)          (xy 111.042702 108.443451)          (xy 111.035004 108.424902)          (xy 111.026401 108.40674)
+          (xy 111.016892 108.388966)          (xy 111.006477 108.371579)          (xy 110.995157 108.35458)          (xy 110.982931 108.337968)
+          (xy 110.9698 108.321743)          (xy 110.955763 108.305905)          (xy 110.940854 108.290709)          (xy 110.925106 108.276493)
+          (xy 110.908519 108.263258)          (xy 110.891094 108.251003)          (xy 110.872829 108.239728)          (xy 110.853726 108.229434)
+          (xy 110.833784 108.22012)          (xy 110.813003 108.211786)          (xy 110.791384 108.204433)          (xy 110.768925 108.198061)
+          (xy 110.745628 108.192668)          (xy 110.721492 108.188257)          (xy 110.696517 108.184825)          (xy 110.670703 108.182374)
+          (xy 110.64405 108.180904)          (xy 110.616559 108.180413)          (xy 110.592273 108.18081)          (xy 110.568655 108.182)
+          (xy 110.545705 108.183984)          (xy 110.523423 108.186761)          (xy 110.501809 108.190331)          (xy 110.480862 108.194695)
+          (xy 110.460583 108.199852)          (xy 110.440973 108.205802)          (xy 110.42203 108.212546)          (xy 110.403755 108.220084)
+          (xy 110.386147 108.228414)          (xy 110.369208 108.237539)          (xy 110.352936 108.247456)          (xy 110.337333 108.258167)
+          (xy 110.322397 108.269672)          (xy 110.308129 108.281969)          (xy 110.294589 108.294915)          (xy 110.281922 108.308363)
+          (xy 110.27013 108.322313)          (xy 110.25921 108.336765)          (xy 110.249164 108.35172)          (xy 110.239992 108.367177)
+          (xy 110.231693 108.383136)          (xy 110.224268 108.399597)          (xy 110.217717 108.41656)          (xy 110.212038 108.434026)
+          (xy 110.207234 108.451994)          (xy 110.203303 108.470464)          (xy 110.200246 108.489436)          (xy 110.198062 108.508911)
+          (xy 110.196751 108.528888)          (xy 110.196315 108.549367)          (xy 110.19661 108.564545)          (xy 110.197495 108.579735)
+          (xy 110.198971 108.594935)          (xy 110.201038 108.610146)          (xy 110.203694 108.625368)          (xy 110.206941 108.6406)
+          (xy 110.210779 108.655843)          (xy 110.215207 108.671097)          (xy 110.220225 108.686362)          (xy 110.225834 108.701637)
+          (xy 110.232033 108.716922)          (xy 110.238822 108.732219)          (xy 110.246202 108.747526)          (xy 110.254172 108.762844)
+          (xy 110.262732 108.778172)          (xy 110.271883 108.793512)          (xy 110.281466 108.80884)          (xy 110.29132 108.824137)
+          (xy 110.301448 108.839401)          (xy 110.311848 108.854633)          (xy 110.32252 108.869834)          (xy 110.333465 108.885002)
+          (xy 110.344682 108.900138)          (xy 110.356172 108.915242)          (xy 110.367934 108.930314)          (xy 110.379968 108.945354)
+          (xy 110.392276 108.960362)          (xy 110.404855 108.975338)          (xy 110.417707 108.990282)          (xy 110.430832 109.005194)
+          (xy 110.444229 109.020074)          (xy 110.457899 109.034921)          (xy 110.831297 109.436017)
         )
       )
@@
     )
   )
-  (gr_text "+" (at 104.9 125.5) (layer "B.SilkS")
-    (effects (font (size 0.8 0.8) (thickness 0.12)) (justify mirror))
-  )
   (gr_text "X32Micro" (at 111.3 107.4) (layer "B.SilkS")
